Commit message: [urdf]: format code for end effectors
Signed-off-by: Jinjie Li <45286479+Li-Jinjie@users.noreply.github.com>

File: robots/beetle_omni/urdf/effectors/ball_ee.xacro (robot description, xacro)
@@ -36,5 +36,5 @@
     <joint name="ee_mount_to_ball" type="fixed">
       <parent link="${ee_mount_link}"/>
-      <child  link="ball"/>
+      <child link="ball"/>
       <origin xyz="0 0 0" rpy="0 0 0"/>
     </joint>
@@ -43,5 +43,5 @@
     <joint name="ball_to_ee_contact" type="fixed">
       <parent link="ball"/>
-      <child  link="ee_contact"/>
+      <child link="ee_contact"/>
       <origin xyz="0 0 0.11" rpy="0 0 0"/>
     </joint>

File: robots/beetle_omni/urdf/effectors/force_sensor_ball_ee.xacro (robot description, xacro)
@@ -38,5 +38,5 @@
     <joint name="ee_mount_to_sensor" type="fixed">
       <parent link="${ee_mount_link}"/>
-      <child  link="wrench_sensor"/>
+      <child link="wrench_sensor"/>
       <origin xyz="0 0 0.031" rpy="0 0 0"/>
     </joint>

File: robots/beetle_omni/urdf/effectors/fork_ee.xacro (robot description, xacro)
@@ -13,6 +13,6 @@
         <mass value="0.140"/>
         <inertia
-                  ixx="0.00040632" iyy="0.00053824" izz="0.00040617"
-                  ixy="0.00000000" ixz="0.00000000" iyz="0.00000000"/>
+                ixx="0.00040632" iyy="0.00053824" izz="0.00040617"
+                ixy="0.00000000" ixz="0.00000000" iyz="0.00000000"/>
       </inertial>
       <visual>
@@ -34,5 +34,5 @@
     <joint name="ee_mount_to_fork" type="fixed">
       <parent link="${ee_mount_link}"/>
-      <child  link="fork"/>
+      <child link="fork"/>
       <origin xyz="0 0 0" rpy="0 0 0"/>
     </joint>
@@ -41,5 +41,5 @@
     <joint name="fork_to_ee_contact" type="fixed">
       <parent link="fork"/>
-      <child  link="ee_contact"/>
+      <child link="ee_contact"/>
       <origin xyz="0 0 0.104" rpy="0 0 0"/>
     </joint>

File: robots/beetle_omni/urdf/effectors/osmo_cam_ee.xacro (robot description, xacro)
@@ -1,97 +1,97 @@
 <?xml version="1.0"?>
 <robot name="osmo_camera_end_effector" xmlns:xacro="http://www.ros.org/wiki/xacro">
-    <!--
-  Macro: osmo_end_effector
-  params:
-    ee_mount_link : The base link connected to the end-effector. (e.g., "ee_mount")
-    robot_ns    : ROS namespace (e.g. "beetle1"). Can be "".
--->
-    <xacro:macro name="osmo_end_effector" params="ee_mount_link robot_ns">
-        <!-- 1) OSMO link and joint -->
-        <link name="osmo">
-            <inertial>
-                <origin xyz="-0.01764 0.02342 0.01321" rpy="0 0 0"/>
-                <mass value="0.1911"/>
-                <inertia
-                        ixx="0.0001070" iyy="0.0001779" izz="0.0001116"
-                        ixy="0.0" ixz="0.0" iyz="0.0"/>
-            </inertial>
-            <visual>
-                <geometry>
-                    <mesh filename="package://beetle_omni/urdf/mesh/end_effector_osmo_camera.dae" scale="1 1 1"/>
-                </geometry>
-            </visual>
-        </link>
-        <joint name="ee_mount_to_osmo" type="fixed">
-            <parent link="${ee_mount_link}"/>
-            <child  link="osmo"/>
-            <origin xyz="0 0 0" rpy="0 0 0"/>
-        </joint>
-        <!-- 2) Attach the reusable camera macro -->
-        <xacro:osmo_rgb_camera parent_link="osmo" robot_ns="${robot_ns}"/>
-        <!-- 3) Contact frame at the bristle tip, required by the outer framework -->
-        <joint name="osmo_to_ee_contact" type="fixed">
-            <parent link="osmo"/>
-            <child link="ee_contact"/>
-            <origin xyz="0 0 0.045" rpy="0 0 0"/>
-        </joint>
-    </xacro:macro>
-    <!--
-      Macro: osmo_rgb_camera
-      params:
-        parent_link : link on which the camera is mounted (e.g. "osmo")
-        robot_ns    : ROS namespace (e.g. "beetle1"). Can be "".
-    -->
-    <xacro:macro name="osmo_rgb_camera" params="parent_link robot_ns">
-        <!-- 1) Optical frame (REP-105): x right, y down, z forward -->
-        <link name="${parent_link}_color_optical_frame"/>
-        <joint name="${parent_link}_color_optical_joint" type="fixed">
-            <parent link="${parent_link}"/>
-            <child  link="${parent_link}_color_optical_frame"/>
-            <!-- lens center offset relative to parent_link -->
-            <origin xyz="0.00 0.00 0.045" rpy="0 -1.570796 0"/>
-        </joint>
-        <!-- 2) Gazebo Classic sensor + ROS plugin -->
-        <gazebo reference="${parent_link}_color_optical_frame">
-            <sensor type="camera" name="${parent_link}_rgb_sensor">
-                <always_on>true</always_on>
-                <update_rate>30</update_rate>
-                <camera name="${parent_link}_rgb">
-                    <!-- hfov from original 3840x2160 calibration -->
-                    <horizontal_fov>1.7663</horizontal_fov>
-                    <image>
-                        <!-- downsampled resolution for faster sim -->
-                        <width>1920</width>
-                        <height>1080</height>
-                        <format>R8G8B8</format>
-                    </image>
-                    <clip>
-                        <near>0.05</near>
-                        <far>50.0</far>
-                    </clip>
-                </camera>
-                <plugin name="${parent_link}_rgb_plugin" filename="libgazebo_ros_camera.so">
-                    <!-- Use robot_ns as ROS namespace, keep cameraName relative -->
-                    <!-- If robot_ns="" this is just the global namespace -->
-                    <robotNamespace>${robot_ns}</robotNamespace>
-                    <frameName>${parent_link}_color_optical_frame</frameName>
-                    <cameraName>osmo/color</cameraName>
-                    <updateRate>30</updateRate>
-                    <!-- Intrinsics scaled for 1920x1080 -->
-                    <focalLength>788.55</focalLength>  <!-- ≈ fx, also used for fy  1577.1 * 0.5 = 788.55 -->
-                    <Cx>961.05</Cx>  <!-- PrincipalPoint(1) 1922.1 * 0.5 = 961.05 -->
-                    <Cy>531.55</Cy>  <!-- PrincipalPoint(2) 1063.1 * 0.5 = 531.55 -->
-                    <!-- Distortion D = [k1 k2 t1 t2 k3] from MATLAB -->
-                    <distortionK1>0.0030</distortionK1>
-                    <distortionK2>-0.0124</distortionK2>
-                    <distortionK3>0.0</distortionK3>
-                    <distortionT1>0.0</distortionT1>
-                    <distortionT2>0.0</distortionT2>
-                    <hackBaseline>0.0</hackBaseline>
-                    <borderCrop>true</borderCrop>
-                    <autoDistortion>false</autoDistortion>
-                </plugin>
-            </sensor>
-        </gazebo>
-    </xacro:macro>
+  <!--
+    Macro: osmo_end_effector
+    params:
+      ee_mount_link : The base link connected to the end-effector. (e.g., "ee_mount")
+      robot_ns    : ROS namespace (e.g. "beetle1"). Can be "".
+  -->
+  <xacro:macro name="osmo_end_effector" params="ee_mount_link robot_ns">
+    <!-- 1) OSMO link and joint -->
+    <link name="osmo">
+      <inertial>
+        <origin xyz="-0.01764 0.02342 0.01321" rpy="0 0 0"/>
+        <mass value="0.1911"/>
+        <inertia
+                ixx="0.0001070" iyy="0.0001779" izz="0.0001116"
+                ixy="0.0" ixz="0.0" iyz="0.0"/>
+      </inertial>
+      <visual>
+        <geometry>
+          <mesh filename="package://beetle_omni/urdf/mesh/end_effector_osmo_camera.dae" scale="1 1 1"/>
+        </geometry>
+      </visual>
+    </link>
+    <joint name="ee_mount_to_osmo" type="fixed">
+      <parent link="${ee_mount_link}"/>
+      <child link="osmo"/>
+      <origin xyz="0 0 0" rpy="0 0 0"/>
+    </joint>
+    <!-- 2) Attach the reusable camera macro -->
+    <xacro:osmo_rgb_camera parent_link="osmo" robot_ns="${robot_ns}"/>
+    <!-- 3) Contact frame at the bristle tip, required by the outer framework -->
+    <joint name="osmo_to_ee_contact" type="fixed">
+      <parent link="osmo"/>
+      <child link="ee_contact"/>
+      <origin xyz="0 0 0.045" rpy="0 0 0"/>
+    </joint>
+  </xacro:macro>
+  <!--
+    Macro: osmo_rgb_camera
+    params:
+      parent_link : link on which the camera is mounted (e.g. "osmo")
+      robot_ns    : ROS namespace (e.g. "beetle1"). Can be "".
+  -->
+  <xacro:macro name="osmo_rgb_camera" params="parent_link robot_ns">
+    <!-- 1) Optical frame (REP-105): x right, y down, z forward -->
+    <link name="${parent_link}_color_optical_frame"/>
+    <joint name="${parent_link}_color_optical_joint" type="fixed">
+      <parent link="${parent_link}"/>
+      <child link="${parent_link}_color_optical_frame"/>
+      <!-- lens center offset relative to parent_link -->
+      <origin xyz="0.00 0.00 0.045" rpy="0 -1.570796 0"/>
+    </joint>
+    <!-- 2) Gazebo Classic sensor + ROS plugin -->
+    <gazebo reference="${parent_link}_color_optical_frame">
+      <sensor type="camera" name="${parent_link}_rgb_sensor">
+        <always_on>true</always_on>
+        <update_rate>30</update_rate>
+        <camera name="${parent_link}_rgb">
+          <!-- hfov from original 3840x2160 calibration -->
+          <horizontal_fov>1.7663</horizontal_fov>
+          <image>
+            <!-- downsampled resolution for faster sim -->
+            <width>1920</width>
+            <height>1080</height>
+            <format>R8G8B8</format>
+          </image>
+          <clip>
+            <near>0.05</near>
+            <far>50.0</far>
+          </clip>
+        </camera>
+        <plugin name="${parent_link}_rgb_plugin" filename="libgazebo_ros_camera.so">
+          <!-- Use robot_ns as ROS namespace, keep cameraName relative -->
+          <!-- If robot_ns="" this is just the global namespace -->
+          <robotNamespace>${robot_ns}</robotNamespace>
+          <frameName>${parent_link}_color_optical_frame</frameName>
+          <cameraName>osmo/color</cameraName>
+          <updateRate>30</updateRate>
+          <!-- Intrinsics scaled for 1920x1080 -->
+          <focalLength>788.55</focalLength>  <!-- ≈ fx, also used for fy  1577.1 * 0.5 = 788.55 -->
+          <Cx>961.05</Cx>  <!-- PrincipalPoint(1) 1922.1 * 0.5 = 961.05 -->
+          <Cy>531.55</Cy>  <!-- PrincipalPoint(2) 1063.1 * 0.5 = 531.55 -->
+          <!-- Distortion D = [k1 k2 t1 t2 k3] from MATLAB -->
+          <distortionK1>0.0030</distortionK1>
+          <distortionK2>-0.0124</distortionK2>
+          <distortionK3>0.0</distortionK3>
+          <distortionT1>0.0</distortionT1>
+          <distortionT2>0.0</distortionT2>
+          <hackBaseline>0.0</hackBaseline>
+          <borderCrop>true</borderCrop>
+          <autoDistortion>false</autoDistortion>
+        </plugin>
+      </sensor>
+    </gazebo>
+  </xacro:macro>
 </robot>
