Commit message: [urdf]: add the geometry part of an ark_flow sensor
Signed-off-by: Jinjie Li <45286479+Li-Jinjie@users.noreply.github.com>

File: robots/beetle_omni/urdf/effectors/brush_ee.xacro (robot description, xacro)
@@ -42,4 +42,45 @@
       <origin xyz="0 0 0.144" rpy="0 0 0"/>
     </joint>
+    <!--  3) Attach the ark_flow_sensor  -->
+    <xacro:ark_flow_sensor parent_link="ee_mount"/>
+  </xacro:macro>
+  <!--
+  Macro: ark_flow_sensor
+  params:
+    parent_link : The link the optical flow sensor attaches to (e.g. "ee_contact").
+-->
+  <xacro:macro name="ark_flow_sensor" params="parent_link">
+    <!-- 1) Optical flow sensor link -->
+    <link name="ark_flow_sensor">
+      <inertial>
+        <!-- Approximate inertial parameters -->
+        <origin xyz="0.0 0.0 0.0" rpy="0 3.141592 0"/>
+        <mass value="0.005"/>
+        <inertia
+                ixx="0.00001" iyy="0.00001" izz="0.00001"
+                ixy="0.0"     ixz="0.0"     iyz="0.0"/>
+      </inertial>
+      <visual>
+        <geometry>
+          <mesh filename="package://beetle_omni/urdf/mesh/ark_flow_mr_rev_1.0.dae"
+                scale="1 1 1"/>
+        </geometry>
+      </visual>
+      <!-- Optional collision -->
+      <!--
+      <collision>
+        <geometry>
+          <mesh filename="package://beetle_omni/urdf/mesh/ark_flow_mr_rev_1.0.dae"
+                scale="1 1 1"/>
+        </geometry>
+      </collision>
+      -->
+    </link>
+    <!-- 2) Fixed joint from parent link to the sensor -->
+    <joint name="ark_flow_sensor_joint" type="fixed">
+      <parent link="${parent_link}"/>
+      <child  link="ark_flow_sensor"/>
+      <origin xyz="-0.08 0 0" rpy="0 0 0"/>
+    </joint>
   </xacro:macro>
 </robot>

Commit message: [urdf]: add optical camera for ark flow sensor
Signed-off-by: Jinjie Li <45286479+Li-Jinjie@users.noreply.github.com>

File: robots/beetle_omni/urdf/effectors/brush_ee.xacro (robot description, xacro)
@@ -50,6 +50,6 @@
     parent_link : The link the optical flow sensor attaches to (e.g. "ee_contact").
 -->
-  <xacro:macro name="ark_flow_sensor" params="parent_link">
-    <!-- 1) Optical flow sensor link -->
+  <xacro:macro name="ark_flow_sensor" params="parent_link robot_ns">
+    <!-- 1) Optical flow sensor link and joint -->
     <link name="ark_flow_sensor">
       <inertial>
@@ -59,5 +59,5 @@
         <inertia
                 ixx="0.00001" iyy="0.00001" izz="0.00001"
-                ixy="0.0"     ixz="0.0"     iyz="0.0"/>
+                ixy="0.0" ixz="0.0" iyz="0.0"/>
       </inertial>
       <visual>
@@ -77,10 +77,40 @@
       -->
     </link>
-    <!-- 2) Fixed joint from parent link to the sensor -->
     <joint name="ark_flow_sensor_joint" type="fixed">
       <parent link="${parent_link}"/>
-      <child  link="ark_flow_sensor"/>
+      <child link="ark_flow_sensor"/>
       <origin xyz="-0.08 0 0" rpy="0 0 0"/>
     </joint>
+    <!-- optical camera -->
+    <link name="optic_cam_link"/>
+    <joint name="optic_cam_joint" type="fixed">
+      <parent link="ark_flow_sensor"/>
+      <child link="optic_cam_link"/>
+      <origin xyz="0.0071 0.00824 0.00154" rpy="0 -1.570796 0"/>  <!-- aim the camera here -->
+    </joint>
+    <gazebo reference="optic_cam_link">
+      <sensor type="camera" name="optic_camera_sensor">
+        <pose>0 0 0 0 0 0</pose>
+        <always_on>true</always_on>
+        <update_rate>50</update_rate>
+        <camera name="optic_rgb">
+          <horizontal_fov>1.047</horizontal_fov>
+          <image>
+            <width>35</width>
+            <height>35</height>
+            <format>R8G8B8</format>
+          </image>
+          <clip>
+            <near>0.08</near>
+            <far>50.0</far>
+          </clip>
+        </camera>
+        <plugin filename="libgazebo_ros_camera.so" name="optic_rgb_plugin">
+          <robotNamespace>${robot_ns}</robotNamespace>
+          <frameName>ark_flow/cam_frame</frameName>
+          <cameraName>ark_flow/cam_color</cameraName>
+        </plugin>
+      </sensor>
+    </gazebo>
   </xacro:macro>
 </robot>

Commit message: [urdf]: refactor the sensors to an independent folder. add ark flow sensor and osmo camera definitions

File: robots/beetle_omni/urdf/effectors/brush_ee.xacro (robot description, xacro)
@@ -45,114 +45,5 @@
     <xacro:ark_flow_sensor parent_link="ee_mount" robot_ns="${robot_ns}"/>
   </xacro:macro>
-  <!--
-  Macro: ark_flow_sensor
-  params:
-    parent_link : The link the optical flow sensor attaches to (e.g. "ee_contact").
--->
-  <xacro:macro name="ark_flow_sensor" params="parent_link robot_ns">
-    <!-- 1) Optical flow sensor link and joint -->
-    <link name="ark_flow_sensor">
-      <inertial>
-        <!-- Approximate inertial parameters -->
-        <origin xyz="0.0 0.0 0.0" rpy="0 3.141592 0"/>
-        <mass value="0.005"/>
-        <inertia
-                ixx="0.00001" iyy="0.00001" izz="0.00001"
-                ixy="0.0" ixz="0.0" iyz="0.0"/>
-      </inertial>
-      <visual>
-        <geometry>
-          <mesh filename="package://beetle_omni/urdf/mesh/ark_flow_mr_rev_1.0.dae"
-                scale="1 1 1"/>
-        </geometry>
-      </visual>
-      <!-- Optional collision -->
-      <!--
-      <collision>
-        <geometry>
-          <mesh filename="package://beetle_omni/urdf/mesh/ark_flow_mr_rev_1.0.dae"
-                scale="1 1 1"/>
-        </geometry>
-      </collision>
-      -->
-    </link>
-    <joint name="ark_flow_sensor_joint" type="fixed">
-      <parent link="${parent_link}"/>
-      <child link="ark_flow_sensor"/>
-      <origin xyz="-0.08 0 0" rpy="0 0 0"/>
-    </joint>
-    <!-- optical camera -->
-    <link name="optic_cam_link"/>
-    <joint name="optic_cam_joint" type="fixed">
-      <parent link="ark_flow_sensor"/>
-      <child link="optic_cam_link"/>
-      <origin xyz="0.0071 0.00824 0.00154" rpy="0 -1.570796 0"/>  <!-- aim the camera here -->
-    </joint>
-    <gazebo reference="optic_cam_link">
-      <sensor type="camera" name="optic_camera_sensor">
-        <pose>0 0 0 0 0 0</pose>
-        <always_on>true</always_on>
-        <update_rate>50</update_rate>
-        <camera name="optic_rgb">
-          <horizontal_fov>1.047</horizontal_fov>
-          <image>
-            <width>35</width>
-            <height>35</height>
-            <format>R8G8B8</format>
-          </image>
-          <clip>
-            <near>0.08</near>
-            <far>50.0</far>
-          </clip>
-        </camera>
-        <plugin filename="libgazebo_ros_camera.so" name="optic_rgb_plugin">
-          <robotNamespace>${robot_ns}</robotNamespace>
-          <frameName>${robot_ns}/optic_cam_link</frameName>
-          <cameraName>ark_flow/cam_color</cameraName>
-        </plugin>
-      </sensor>
-    </gazebo>
-    <!-- point laser -->
-    <!-- the frame of point laser is aligned with optic_cam_link for simplicity -->
-    <gazebo reference="optic_cam_link">
-      <sensor type="ray" name="point_laser_sensor">
-        <pose>0 0 0 0 0 0</pose>
-        <always_on>true</always_on>
-        <update_rate>100</update_rate>
-        <ray>
-          <scan>
-            <horizontal>
-              <samples>1</samples>
-              <resolution>1</resolution>
-              <min_angle>0</min_angle>
-              <max_angle>0</max_angle>
-            </horizontal>
-            <vertical>
-              <samples>1</samples>
-              <resolution>1</resolution>
-              <min_angle>0.0</min_angle>
-              <max_angle>0.0</max_angle>
-            </vertical>
-          </scan>
-          <range>
-            <min>0.02</min>
-            <max>10.0</max>
-          </range>
-        </ray>
-        <!--        <noise>-->
-        <!--          <type>gaussian</type>-->
-        <!--          <mean>0.0</mean>-->
-        <!--          <stddev>0.005</stddev>-->
-        <!--        </noise>-->
-        <plugin filename="libgazebo_ros_range.so" name="point_laser_plugin">
-          <!-- ATTENTION: here are topicName and frameName, not topic_name! -->
-          <robotNamespace>${robot_ns}</robotNamespace>
-          <frameName>${robot_ns}/optic_cam_link</frameName>
-          <topicName>ark_flow/point_laser</topicName>
-          <!-- radiation_type：0=ULTRASOUND，1=INFRARED -->
-          <radiation_type>1</radiation_type>
-        </plugin>
-      </sensor>
-    </gazebo>
-  </xacro:macro>
+  <!-- include shared sensors -->
+  <xacro:include filename="$(find beetle_omni)/urdf/sensors/ark_flow.xacro"/>
 </robot>

File: robots/beetle_omni/urdf/effectors/osmo_cam_ee.xacro (robot description, xacro)
@@ -37,61 +37,5 @@
     </joint>
   </xacro:macro>
-  <!--
-    Macro: osmo_rgb_camera
-    params:
-      parent_link : link on which the camera is mounted (e.g. "osmo")
-      robot_ns    : ROS namespace (e.g. "beetle1"). Can be "".
-  -->
-  <xacro:macro name="osmo_rgb_camera" params="parent_link robot_ns">
-    <!-- 1) Optical frame (REP-105): x right, y down, z forward -->
-    <link name="${parent_link}_color_optical_frame"/>
-    <joint name="${parent_link}_color_optical_joint" type="fixed">
-      <parent link="${parent_link}"/>
-      <child link="${parent_link}_color_optical_frame"/>
-      <!-- lens center offset relative to parent_link -->
-      <origin xyz="0.00 0.00 0.045" rpy="0 -1.570796 0"/>
-    </joint>
-    <!-- 2) Gazebo Classic sensor + ROS plugin -->
-    <gazebo reference="${parent_link}_color_optical_frame">
-      <sensor type="camera" name="${parent_link}_rgb_sensor">
-        <always_on>true</always_on>
-        <update_rate>30</update_rate>
-        <camera name="${parent_link}_rgb">
-          <!-- hfov from original 3840x2160 calibration -->
-          <horizontal_fov>1.7663</horizontal_fov>
-          <image>
-            <!-- downsampled resolution for faster sim -->
-            <width>1920</width>
-            <height>1080</height>
-            <format>R8G8B8</format>
-          </image>
-          <clip>
-            <near>0.05</near>
-            <far>50.0</far>
-          </clip>
-        </camera>
-        <plugin name="${parent_link}_rgb_plugin" filename="libgazebo_ros_camera.so">
-          <!-- Use robot_ns as ROS namespace, keep cameraName relative -->
-          <!-- If robot_ns="" this is just the global namespace -->
-          <robotNamespace>${robot_ns}</robotNamespace>
-          <frameName>${robot_ns}/${parent_link}_color_optical_frame</frameName>
-          <cameraName>osmo/color</cameraName>
-          <updateRate>30</updateRate>
-          <!-- Intrinsics scaled for 1920x1080 -->
-          <focalLength>788.55</focalLength>  <!-- ≈ fx, also used for fy  1577.1 * 0.5 = 788.55 -->
-          <Cx>961.05</Cx>  <!-- PrincipalPoint(1) 1922.1 * 0.5 = 961.05 -->
-          <Cy>531.55</Cy>  <!-- PrincipalPoint(2) 1063.1 * 0.5 = 531.55 -->
-          <!-- Distortion D = [k1 k2 t1 t2 k3] from MATLAB -->
-          <distortionK1>0.0030</distortionK1>
-          <distortionK2>-0.0124</distortionK2>
-          <distortionK3>0.0</distortionK3>
-          <distortionT1>0.0</distortionT1>
-          <distortionT2>0.0</distortionT2>
-          <hackBaseline>0.0</hackBaseline>
-          <borderCrop>true</borderCrop>
-          <autoDistortion>false</autoDistortion>
-        </plugin>
-      </sensor>
-    </gazebo>
-  </xacro:macro>
+  <!-- include shared sensors -->
+  <xacro:include filename="$(find beetle_omni)/urdf/sensors/osmo_camera.xacro"/>
 </robot>

Commit message: [urdf]: enhance ark flow sensor definition with additional parameters for name, supporting the case for multiple sensors.

File: robots/beetle_omni/urdf/effectors/brush_ee.xacro (robot description, xacro)
@@ -43,5 +43,5 @@
     </joint>
     <!--  3) Attach the ark_flow_sensor  -->
-    <xacro:ark_flow_sensor parent_link="ee_mount" robot_ns="${robot_ns}"/>
+    <xacro:ark_flow_sensor name="ark_flow" parent_link="ee_mount" robot_ns="${robot_ns}"/>
   </xacro:macro>
   <!-- include shared sensors -->

File: robots/beetle_omni/urdf/sensors/ark_flow.xacro (robot description, xacro)
@@ -4,9 +4,13 @@
   Macro: ark_flow_sensor
   params:
-    parent_link : The link the optical flow sensor attaches to (e.g. "ee_contact").
+    name        : Unique name/prefix for this sensor instance (e.g. "ark_flow_1", "ark_flow_2").
+    parent_link : The link the optical flow sensor attaches to (e.g. "ee_mount").
+    robot_ns    : ROS namespace (e.g. "beetle1"). Can be "".
+    xyz         : Position offset relative to parent_link (default: "-0.08 0 0").
+    rpy         : Orientation offset relative to parent_link (default: "0 0 0").
   -->
-  <xacro:macro name="ark_flow_sensor" params="parent_link robot_ns">
+  <xacro:macro name="ark_flow_sensor" params="name parent_link robot_ns xyz:='-0.08 0 0' rpy:='0 0 0'">
     <!-- 1) Optical flow sensor link and joint -->
-    <link name="ark_flow_sensor">
+    <link name="${name}">
       <inertial>
         <!-- Approximate inertial parameters -->
@@ -33,22 +37,22 @@
       -->
     </link>
-    <joint name="ark_flow_sensor_joint" type="fixed">
+    <joint name="${name}_joint" type="fixed">
       <parent link="${parent_link}"/>
-      <child link="ark_flow_sensor"/>
-      <origin xyz="-0.08 0 0" rpy="0 0 0"/>
+      <child link="${name}"/>
+      <origin xyz="${xyz}" rpy="${rpy}"/>
     </joint>
     <!-- optical camera -->
-    <link name="optic_cam_link"/>
-    <joint name="optic_cam_joint" type="fixed">
-      <parent link="ark_flow_sensor"/>
-      <child link="optic_cam_link"/>
+    <link name="${name}_optic_cam"/>
+    <joint name="${name}_optic_cam_joint" type="fixed">
+      <parent link="${name}"/>
+      <child link="${name}_optic_cam"/>
       <origin xyz="0.0071 0.00824 0.00154" rpy="0 -1.570796 0"/>  <!-- aim the camera here -->
     </joint>
-    <gazebo reference="optic_cam_link">
-      <sensor type="camera" name="optic_camera_sensor">
+    <gazebo reference="${name}_optic_cam">
+      <sensor type="camera" name="${name}_optic_camera_sensor">
         <pose>0 0 0 0 0 0</pose>
         <always_on>true</always_on>
         <update_rate>50</update_rate>
-        <camera name="optic_rgb">
+        <camera name="${name}_optic_rgb">
           <horizontal_fov>1.047</horizontal_fov>
           <image>
@@ -62,15 +66,15 @@
           </clip>
         </camera>
-        <plugin filename="libgazebo_ros_camera.so" name="optic_rgb_plugin">
+        <plugin filename="libgazebo_ros_camera.so" name="${name}_optic_rgb_plugin">
           <robotNamespace>${robot_ns}</robotNamespace>
-          <frameName>${robot_ns}/optic_cam_link</frameName>
-          <cameraName>ark_flow/cam_color</cameraName>
+          <frameName>${robot_ns}/${name}_optic_cam</frameName>
+          <cameraName>${name}/cam_color</cameraName>
         </plugin>
       </sensor>
     </gazebo>
     <!-- point laser -->
-    <!-- the frame of point laser is aligned with optic_cam_link for simplicity -->
-    <gazebo reference="optic_cam_link">
-      <sensor type="ray" name="point_laser_sensor">
+    <!-- the frame of point laser is aligned with optic_cam for simplicity -->
+    <gazebo reference="${name}_optic_cam">
+      <sensor type="ray" name="${name}_point_laser_sensor">
         <pose>0 0 0 0 0 0</pose>
         <always_on>true</always_on>
@@ -101,9 +105,9 @@
         <!--          <stddev>0.005</stddev>-->
         <!--        </noise>-->
-        <plugin filename="libgazebo_ros_range.so" name="point_laser_plugin">
+        <plugin filename="libgazebo_ros_range.so" name="${name}_point_laser_plugin">
           <!-- ATTENTION: here are topicName and frameName, not topic_name! -->
           <robotNamespace>${robot_ns}</robotNamespace>
-          <frameName>${robot_ns}/optic_cam_link</frameName>
-          <topicName>ark_flow/point_laser</topicName>
+          <frameName>${robot_ns}/${name}_optic_cam</frameName>
+          <topicName>${name}/point_laser</topicName>
           <!-- radiation_type：0=ULTRASOUND，1=INFRARED -->
           <radiation_type>1</radiation_type>
