Commit message: [urdf][beetle-omni]: remove common.xacro and put contents into one urdf.
Signed-off-by: LI, Jinjie <li-jinjie@g.ecc.u-tokyo.ac.jp>

File: robots/beetle_omni/robots/beetle_art_omni.urdf.xacro (robot description, xacro)
@@ -1,5 +1,4 @@
 <?xml version="1.0"?>
 <robot xmlns:xacro="http://www.ros.org/wiki/xacro" name="beetle-art-omni" >
-  <xacro:include filename="$(find beetle_omni)/urdf/common.xacro" />
   <xacro:include filename="$(find beetle_omni)/urdf/beetle_art_omni.urdf.xacro" />
 </robot>

File: robots/beetle_omni/urdf/beetle_art_omni.urdf.xacro (robot description, xacro)
@@ -1,4 +1,23 @@
 <?xml version="1.0"?>
 <robot xmlns:xacro="http://www.ros.org/wiki/xacro" name="beetle_link" >
+  <!-- general attribute -->
+  <baselink name="fc" />
+  <thrust_link name="thrust" />
+  <m_f_rate value="-0.0165" /> <!-- drag torque rate -->
+  <xacro:property name="max_force" value="30.0" /> <!-- [N] -->
+  <xacro:property name="min_force" value="1.0" /> <!-- [N] -->
+  <!-- friction -->
+  <xacro:macro name="friction" params="self">
+    <gazebo reference="link${self}">
+      <mu1>0.1</mu1>
+      <mu2>0.1</mu2>
+    </gazebo>
+  </xacro:macro>
+  <xacro:macro name="damping_factor" params="link">
+    <gazebo reference="${link}">
+      <dampingFactor>0.00</dampingFactor>
+    </gazebo>
+  </xacro:macro>
+  <!-- robot -->
   <xacro:macro name="beetle_center_link" params="child1 child2 child3 child4">
     ## dummy
@@ -31,5 +50,4 @@
       <origin rpy="0 0 0" xyz="0 0 0"/>
     </joint>
-    ## fc: flight controller. Note that "baselink" is assigned to "fc" in common.xacro by default
     <link name="fc">
       <inertial>
