Commit message: [urdf][dragon-ball]: init the URDF of dragon_ball
Signed-off-by: LI, Jinjie <li-jinjie@g.ecc.u-tokyo.ac.jp>

File: robots/beetle_omni/robots/dragon_ball.urdf.xacro (robot description, xacro)
@@ -1,4 +1,4 @@
 <?xml version="1.0"?>
 <robot xmlns:xacro="http://www.ros.org/wiki/xacro" name="dragon-ball" >
-  <xacro:include filename="$(find beetle_omni)/urdf/dragon-ball.urdf.xacro" />
+  <xacro:include filename="$(find beetle_omni)/urdf/dragon_ball.urdf.xacro" />
 </robot>

File: robots/beetle_omni/urdf/dragon_ball.urdf.xacro (robot description, xacro)
@@ -26,20 +26,20 @@
     <link name="main_body">
       <inertial>
-        <origin xyz="- 0.00023741 0.01491666" rpy="0 0 0"/>
-        <mass value="2.27739"/>
-        <inertia
-            ixx="0.02747704" iyy="0.02676088" izz="0.04047304"
-            ixy="-0.00000599" ixz="0.00009626" iyz="0.00006750"/>
+        <origin xyz="-0.00058556 0.00011136 0.00444799" rpy="0 0 0"/>
+        <mass value="1.1340"/>
+        <inertia
+            ixx="0.00358514" iyy="0.00354587" izz="0.00357606"
+            ixy="-0.00000033" ixz="-0.00005534" iyz="0.00000798"/>
       </inertial>
       <visual>
         <origin xyz="0 0 0" rpy="0 0 0"/>
         <geometry>
-          <mesh filename="package://beetle_omni/urdf/mesh/main_body_beetle_omni_w_guard.dae"/>
+          <mesh filename="package://beetle_omni/urdf/mesh/center_module_dragon_ball.dae"/>
         </geometry>
       </visual>
       <collision>
-        <origin xyz="0 0 0.0385" rpy="0 0 0"/>
-        <geometry>
-          <box size="0.35 0.35 0.275"/>
+        <origin xyz="0 0 0.021" rpy="0 0 0"/>
+        <geometry>
+          <box size="0.15 0.15 0.160"/>
         </geometry>
       </collision>
@@ -63,5 +63,5 @@
       <child link="fc"/>
       <parent link="main_body"/>
-      <origin rpy="0 0 0" xyz="-0.0175 -0.0015 0.06647"/>  # should be aligned with the position of IMU
+      <origin rpy="0 0 0" xyz="-0.0175 -0.0015 0.075"/>  # should be aligned with the position of IMU
     </joint>
     ## rotor arm macro
@@ -86,8 +86,8 @@
     </xacro:macro>
     ## dummy rotor arms
-    <xacro:dummy_rotor_arm id = "${child1}" x = "0.17938" y="0.17938" z = "0.0171" yaw = "${pi*1.0/4.0}"/>
-    <xacro:dummy_rotor_arm id = "${child2}" x = "-0.17938" y="0.17938" z = "0.0171" yaw = "${pi*3.0/4.0}"/>
-    <xacro:dummy_rotor_arm id = "${child3}" x = "-0.17938" y="-0.17938" z = "0.0171" yaw = "${pi*5.0/4.0}"/>
-    <xacro:dummy_rotor_arm id = "${child4}" x = "0.17938" y="-0.17938" z = "0.0171" yaw = "${-pi*1.0/4.0}"/>
+    <xacro:dummy_rotor_arm id = "${child1}" x = "0.08231" y="0.08231" z = "0.0175" yaw = "${pi*1.0/4.0}"/>
+    <xacro:dummy_rotor_arm id = "${child2}" x = "-0.08231" y="0.08231" z = "0.0175" yaw = "${pi*3.0/4.0}"/>
+    <xacro:dummy_rotor_arm id = "${child3}" x = "-0.08231" y="-0.08231" z = "0.0175" yaw = "${pi*5.0/4.0}"/>
+    <xacro:dummy_rotor_arm id = "${child4}" x = "0.08231" y="-0.08231" z = "0.0175" yaw = "${-pi*1.0/4.0}"/>
     <xacro:friction self="main_body"/>
   </xacro:macro>
@@ -97,14 +97,14 @@
     <link name="gimbal_link${self}">
       <inertial>
-        <origin xyz="0.02085225 0.0 -0.01276312" rpy="0 0 0"/>
-        <mass value="0.15944"/>
-        <inertia
-            ixx="0.00007281" iyy="0.00007289" izz="0.00007635"
-            ixy="0.0" ixz="0.0" iyz="0.0"/>
+        <origin xyz="0.01809124 0.0 -0.02799847" rpy="0 0 0"/>
+        <mass value="0.065"/>
+        <inertia
+            ixx="0.00003763" iyy="0.00003471" izz="0.00005131"
+            ixy="0.0" ixz="-0.00000255" iyz="0.0"/>
       </inertial>
       <collision>
-        <origin xyz="0.06 0 0" rpy="0 0 0"/>
-        <geometry>
-          <box size="0.11 0.11 0.05"/>
+        <origin xyz="0.06 0 -0.03" rpy="0 0 0"/>
+        <geometry>
+          <box size="0.08 0.13 0.043"/>
         </geometry>
       </collision>
@@ -112,5 +112,5 @@
         <origin xyz="0 0 0" rpy="0 0 0"/>
         <geometry>
-          <mesh filename="package://beetle_omni/urdf/mesh/omni_rotor_module.dae"/>
+          <mesh filename="package://beetle_omni/urdf/mesh/omni_rotor_module_5inch.dae"/>
         </geometry>
       </visual>
@@ -164,5 +164,5 @@
       <parent link="gimbal_link${self}"/>
       <child link="rotor_parent${self}"/>
-      <origin rpy="0 0 0" xyz="0.02185 0.0 0.0"/>
+      <origin rpy="0 0 0" xyz="0.0 0.0 0.0"/>
     </joint>
     #### rotor joint (virtual) ####
@@ -206,5 +206,5 @@
     <parent link="main_body"/>
     <child link="ee_mount"/>
-    <origin xyz="0 0 0.1725" rpy="0 0 0"/>
+    <origin xyz="0 0 0.104" rpy="0 0 0"/>
   </joint>
   <!-- Tool‑agnostic contact frame (pose set inside each branch) -->
