Commit message: [beetle-omni] update the physical parameters for beetle-omni with a fork-like end effector

File: robots/beetle_omni/urdf/beetle_art_omni.urdf.xacro (robot description, xacro)
@@ -7,9 +7,9 @@
     <link name="main_body">
       <inertial>
-        <origin xyz="0.00000845 0.00023419 0.02260762" rpy="0 0 0"/>
-        <mass value="2.3096"/>
+        <origin xyz="0.00001134 0.00022365 0.02791215" rpy="0 0 0"/>
+        <mass value="2.4173"/>
         <inertia
-            ixx="0.03155716" iyy="0.03084096" izz="0.03900553"
-            ixy="-0.00000599" ixz="0.00008620" iyz="0.00005548"/>
+            ixx="0.03452434" iyy="0.03380832" izz="0.04101129"
+            ixy="-0.00000600" ixz="0.00009772" iyz="0.00006047"/>
       </inertial>
       <visual>

Commit message: [robot]: add urdf for an effector to mount osmo action 4

File: robots/beetle_omni/urdf/beetle_art_omni.urdf.xacro (robot description, xacro)
@@ -323,3 +323,31 @@
     </joint>
   </xacro:if>
+  <!-- ############# DJI OSMO Action 4 ############# -->
+  <xacro:if value="${end_effector == 'osmo'}">
+    <link name="osmo">
+      <inertial>
+        <origin xyz="-0.01764 0.02342 0.01321" rpy="0 0 0"/>
+        <mass value="0.1911"/>
+        <inertia
+                ixx="0.0001070" iyy="0.0001779" izz="0.0001116"
+                ixy="-0.000000" ixz="0.00000000" iyz="0.00000000"/>
+      </inertial>
+      <visual>
+        <geometry>
+          <mesh filename="package://beetle_omni/urdf/mesh/end_effector_osmo_camera.dae" scale="1 1 1"/>
+        </geometry>
+      </visual>
+    </link>
+    <joint name="ee_mount_to_osmo" type="fixed">
+      <parent link="ee_mount"/>
+      <child link="osmo"/>
+      <origin xyz="0 0 0" rpy="0 0 0"/>
+    </joint>
+    <!-- Contact frame at the bristle tip -->
+    <joint name="osmo_to_ee_contact" type="fixed">
+      <parent link="osmo"/>
+      <child link="ee_contact"/>
+      <origin xyz="0 0 0.045" rpy="0 0 0"/>
+    </joint>
+  </xacro:if>
 </robot>

Commit message: [urdf]: add the camera model to the URDF file for the osmo camera.

File: robots/beetle_omni/urdf/beetle_art_omni.urdf.xacro (robot description, xacro)
@@ -325,4 +325,49 @@
   <!-- ############# DJI OSMO Action 4 ############# -->
   <xacro:if value="${end_effector == 'osmo'}">
+    <!-- Contact frame at the bristle tip, required by the outer framework -->
+    <joint name="osmo_to_ee_contact" type="fixed">
+      <parent link="osmo"/>
+      <child link="ee_contact"/>
+      <origin xyz="0 0 0.045" rpy="0 0 0"/>
+    </joint>
+    <!-- 1) Optical frame (REP-105): x right, y down, z forward -->
+    <!-- Tip: move xyz to the actual lens center relative to the 'osmo' link -->
+    <link name="osmo_color_optical_frame"/>
+    <joint name="osmo_color_optical_joint" type="fixed">
+      <parent link="osmo"/>
+      <child  link="osmo_color_optical_frame"/>
+      <origin xyz="0.00 0.00 0.045" rpy="3.141593 -1.570796 0"/>
+    </joint>
+    <!-- 2) Gazebo Classic sensor + ROS plugin -->
+    <gazebo reference="osmo_color_optical_frame">
+      <sensor type="camera" name="osmo_rgb_sensor">
+        <!-- The pose of camera must be independently set, better align to osmo_color_optical_frame -->
+        <always_on>true</always_on>
+        <update_rate>30</update_rate>
+        <camera name="osmo_rgb">
+          <!-- Horizontal FOV and intrinsics: adjust as you like -->
+          <horizontal_fov>1.047</horizontal_fov> <!-- ~60 deg -->
+          <image>
+            <width>1280</width>
+            <height>720</height>
+            <format>R8G8B8</format>
+          </image>
+          <clip>
+            <near>0.05</near>
+            <far>50.0</far>
+          </clip>
+        </camera>
+        <plugin name="osmo_rgb_plugin" filename="libgazebo_ros_camera.so">
+          <ros>
+            <namespace>/</namespace>
+          </ros>
+          <frame_name>osmo_color_optical_frame</frame_name>
+          <camera_name>osmo/color</camera_name>
+          <hack_baseline>0.0</hack_baseline>
+          <publish_rate>30</publish_rate>
+        </plugin>
+      </sensor>
+    </gazebo>
+    <!-- 3) OSMO link and joints -->
     <link name="osmo">
       <inertial>
@@ -344,10 +389,4 @@
       <origin xyz="0 0 0" rpy="0 0 0"/>
     </joint>
-    <!-- Contact frame at the bristle tip -->
-    <joint name="osmo_to_ee_contact" type="fixed">
-      <parent link="osmo"/>
-      <child link="ee_contact"/>
-      <origin xyz="0 0 0.045" rpy="0 0 0"/>
-    </joint>
   </xacro:if>
 </robot>

Commit message: [urdf][osmo]: correct the direction of camera

File: robots/beetle_omni/urdf/beetle_art_omni.urdf.xacro (robot description, xacro)
@@ -337,5 +337,5 @@
       <parent link="osmo"/>
       <child  link="osmo_color_optical_frame"/>
-      <origin xyz="0.00 0.00 0.045" rpy="3.141593 -1.570796 0"/>
+      <origin xyz="0.00 0.00 0.045" rpy="0 -1.570796 0"/>
     </joint>
     <!-- 2) Gazebo Classic sensor + ROS plugin -->

Commit message: [beetle-omni][urdf]: ATTENTION: the arg must be used together with property!!!!!! Otherwise the ${} notation cannot work.

File: robots/beetle_omni/urdf/beetle_art_omni.urdf.xacro (robot description, xacro)
@@ -169,4 +169,5 @@
 <!-- Define beetle -->
   <xacro:arg name="robot_name" default="beetle-art-omni" />
+  <xacro:property name="robot_name" value="$(arg robot_name)"/>
   <xacro:beetle_center_link child1="1" child2="2" child3="3" child4="4"/>
   <xacro:beetle_thrust_link self="1" rotor_direction="1"/>

Commit message: [beetle-omni][urdf]: separate one osmo camera into an additional urdf file.

File: robots/beetle_omni/urdf/beetle_art_omni.urdf.xacro (robot description, xacro)
@@ -325,4 +325,5 @@
   </xacro:if>
   <!-- ############# DJI OSMO Action 4 ############# -->
+  <xacro:include filename="$(find beetle_omni)/urdf/osmo_camera.xacro"/>
   <xacro:if value="${end_effector == 'osmo'}">
     <!-- Contact frame at the bristle tip, required by the outer framework -->
@@ -332,52 +333,4 @@
       <origin xyz="0 0 0.045" rpy="0 0 0"/>
     </joint>
-    <!-- 1) Optical frame (REP-105): x right, y down, z forward -->
-    <!-- Tip: move xyz to the actual lens center relative to the 'osmo' link -->
-    <link name="osmo_color_optical_frame"/>
-    <joint name="osmo_color_optical_joint" type="fixed">
-      <parent link="osmo"/>
-      <child  link="osmo_color_optical_frame"/>
-      <origin xyz="0.00 0.00 0.045" rpy="0 -1.570796 0"/>
-    </joint>
-    <!-- 2) Gazebo Classic sensor + ROS plugin -->
-    <gazebo reference="osmo_color_optical_frame">
-      <sensor type="camera" name="osmo_rgb_sensor">
-        <!-- The pose of camera must be independently set, better align to osmo_color_optical_frame -->
-        <always_on>true</always_on>
-        <update_rate>30</update_rate>
-        <camera name="osmo_rgb">
-          <!-- Horizontal FOV and intrinsics: adjust as you like -->
-          <horizontal_fov>1.7663</horizontal_fov> <!-- 2 arctan (3840 / (2 * 1577.1)) -->
-          <image>
-          <!--  original: 2160 * 3840-->
-            <width>1920</width>
-            <height>1080</height>
-            <format>R8G8B8</format>
-          </image>
-          <clip>
-            <near>0.05</near>
-            <far>50.0</far>
-          </clip>
-        </camera>
-        <plugin name="osmo_rgb_plugin" filename="libgazebo_ros_camera.so">
-          <frameName>osmo_color_optical_frame</frameName>
-          <cameraName>osmo/color</cameraName>
-          <updateRate>30</updateRate>
-          <focalLength>788.55</focalLength>      <!-- ≈ fx, also used for fy  1577.1 * 0.5 = 788.55 -->
-          <Cx>961.05</Cx>                        <!-- PrincipalPoint(1) 1922.1 * 0.5 = 961.05 -->
-          <Cy>531.55</Cy>                        <!-- PrincipalPoint(2) 1063.1 * 0.5 = 531.55 -->
-          <!-- Distortion D = [k1 k2 t1 t2 k3] -->
-          <distortionK1>0.0030</distortionK1>    <!-- RadialDistortion(1) -->
-          <distortionK2>-0.0124</distortionK2>   <!-- RadialDistortion(2) -->
-          <distortionK3>0.0</distortionK3>       <!-- no k3 from MATLAB -->
-          <distortionT1>0.0</distortionT1>       <!-- TangentialDistortion(1) -->
-          <distortionT2>0.0</distortionT2>       <!-- TangentialDistortion(2) -->
-          <!-- Optional extras -->
-          <hackBaseline>0.0</hackBaseline>       <!-- non-stereo -->
-          <borderCrop>true</borderCrop>          <!-- default behavior -->
-          <autoDistortion>false</autoDistortion> <!-- use above coefficients -->
-        </plugin>
-      </sensor>
-    </gazebo>
     <!-- 3) OSMO link and joints -->
     <link name="osmo">
@@ -387,5 +340,5 @@
         <inertia
                 ixx="0.0001070" iyy="0.0001779" izz="0.0001116"
-                ixy="-0.000000" ixz="0.00000000" iyz="0.00000000"/>
+                ixy="0.0" ixz="0.0" iyz="0.0"/>
       </inertial>
       <visual>
@@ -400,4 +353,6 @@
       <origin xyz="0 0 0" rpy="0 0 0"/>
     </joint>
+    <!-- 4) Attach the reusable camera macro -->
+    <xacro:osmo_rgb_camera parent_link="osmo" robot_ns="${robot_name}"/>
   </xacro:if>
 </robot>

Commit message: [urdf]: refactor osmo_cam_ee.xacro and put most contents from the main file into it

File: robots/beetle_omni/urdf/beetle_art_omni.urdf.xacro (robot description, xacro)
@@ -331,32 +331,5 @@
   <xacro:include filename="$(find beetle_omni)/urdf/effectors/osmo_cam_ee.xacro"/>
   <xacro:if value="${end_effector == 'osmo'}">
-    <!-- Contact frame at the bristle tip, required by the outer framework -->
-    <joint name="osmo_to_ee_contact" type="fixed">
-      <parent link="osmo"/>
-      <child link="ee_contact"/>
-      <origin xyz="0 0 0.045" rpy="0 0 0"/>
-    </joint>
-    <!-- 3) OSMO link and joints -->
-    <link name="osmo">
-      <inertial>
-        <origin xyz="-0.01764 0.02342 0.01321" rpy="0 0 0"/>
-        <mass value="0.1911"/>
-        <inertia
-                ixx="0.0001070" iyy="0.0001779" izz="0.0001116"
-                ixy="0.0" ixz="0.0" iyz="0.0"/>
-      </inertial>
-      <visual>
-        <geometry>
-          <mesh filename="package://beetle_omni/urdf/mesh/end_effector_osmo_camera.dae" scale="1 1 1"/>
-        </geometry>
-      </visual>
-    </link>
-    <joint name="ee_mount_to_osmo" type="fixed">
-      <parent link="ee_mount"/>
-      <child link="osmo"/>
-      <origin xyz="0 0 0" rpy="0 0 0"/>
-    </joint>
-    <!-- 4) Attach the reusable camera macro -->
-    <xacro:osmo_rgb_camera parent_link="osmo" robot_ns="${robot_name}"/>
+    <xacro:osmo_end_effector ee_mount_link="ee_mount" robot_ns="${robot_name}"/>
   </xacro:if>
 </robot>

File: robots/beetle_omni/urdf/effectors/osmo_cam_ee.xacro (robot description, xacro)
@@ -1,4 +1,40 @@
 <?xml version="1.0"?>
-<robot name="osmo_camera" xmlns:xacro="http://www.ros.org/wiki/xacro">
+<robot name="osmo_camera_end_effector" xmlns:xacro="http://www.ros.org/wiki/xacro">
+    <!--
+  Macro: osmo_end_effector
+  params:
+    ee_mount_link : The base link connected to the end-effector. (e.g., "ee_mount")
+    robot_ns    : ROS namespace (e.g. "beetle1"). Can be "".
+-->
+    <xacro:macro name="osmo_end_effector" params="ee_mount_link robot_ns">
+        <!-- 1) OSMO link and joint -->
+        <link name="osmo">
+            <inertial>
+                <origin xyz="-0.01764 0.02342 0.01321" rpy="0 0 0"/>
+                <mass value="0.1911"/>
+                <inertia
+                        ixx="0.0001070" iyy="0.0001779" izz="0.0001116"
+                        ixy="0.0" ixz="0.0" iyz="0.0"/>
+            </inertial>
+            <visual>
+                <geometry>
+                    <mesh filename="package://beetle_omni/urdf/mesh/end_effector_osmo_camera.dae" scale="1 1 1"/>
+                </geometry>
+            </visual>
+        </link>
+        <joint name="ee_mount_to_osmo" type="fixed">
+            <parent link="${ee_mount_link}"/>
+            <child  link="osmo"/>
+            <origin xyz="0 0 0" rpy="0 0 0"/>
+        </joint>
+        <!-- 2) Attach the reusable camera macro -->
+        <xacro:osmo_rgb_camera parent_link="osmo" robot_ns="${robot_ns}"/>
+        <!-- 3) Contact frame at the bristle tip, required by the outer framework -->
+        <joint name="osmo_to_ee_contact" type="fixed">
+            <parent link="osmo"/>
+            <child link="ee_contact"/>
+            <origin xyz="0 0 0.045" rpy="0 0 0"/>
+        </joint>
+    </xacro:macro>
     <!--
       Macro: osmo_rgb_camera

Commit message: [urdf]: create brush_ee.xacro and put most contents from the main file into it

File: robots/beetle_omni/urdf/beetle_art_omni.urdf.xacro (robot description, xacro)
@@ -301,30 +301,7 @@
   </xacro:if>
   <!-- ############# Brush tool ############# -->
+  <xacro:include filename="$(find beetle_omni)/urdf/effectors/brush_ee.xacro"/>
   <xacro:if value="${end_effector == 'brush'}">
-    <link name="brush">
-      <inertial>
-        <origin xyz="0.00000000 0.06565796 -0.00001172" rpy="0 0 0"/>
-        <mass value="0.100"/>
-        <inertia
-                ixx="0.00019687" iyy="0.00013173" izz="0.00019689"
-                ixy="0.00000000" ixz="0.00000000" iyz="0.00000000"/>
-      </inertial>
-      <visual>
-        <geometry>
-          <mesh filename="package://beetle_omni/urdf/mesh/end_effector_brush.dae" scale="1 1 1"/>
-        </geometry>
-      </visual>
-    </link>
-    <joint name="ee_mount_to_brush" type="fixed">
-      <parent link="ee_mount"/>
-      <child link="brush"/>
-      <origin xyz="0 0 0" rpy="0 0 0"/>
-    </joint>
-    <!-- Contact frame at the bristle tip -->
-    <joint name="brush_to_ee_contact" type="fixed">
-      <parent link="brush"/>
-      <child link="ee_contact"/>
-      <origin xyz="0 0 0.144" rpy="0 0 0"/>
-    </joint>
+    <xacro:brush_end_effector ee_mount_link="ee_mount"/>
   </xacro:if>
   <!-- ############# DJI OSMO Action 4 ############# -->

Commit message: [urdf]: create fork_ee.xacro and put most contents from the main file into it
Signed-off-by: Jinjie Li <45286479+Li-Jinjie@users.noreply.github.com>

File: robots/beetle_omni/urdf/beetle_art_omni.urdf.xacro (robot description, xacro)
@@ -193,32 +193,7 @@
   <link name="ee_contact"/>
   <!-- ############# Fork tool ############# -->
+  <xacro:include filename="$(find beetle_omni)/urdf/effectors/fork_ee.xacro"/>
   <xacro:if value="${end_effector == 'fork'}">
-    <!-- Tool geometry -->
-    <link name="fork">
-      <inertial>
-        <origin xyz="0.00000000 0.06681059 -0.00005783" rpy="0 0 0"/>
-        <mass value="0.140"/>
-        <inertia
-                ixx="0.00040632" iyy="0.00053824" izz="0.00040617"
-                ixy="0.00000000" ixz="0.00000000" iyz="0.00000000"/>
-      </inertial>
-      <visual>
-        <geometry>
-          <mesh filename="package://beetle_omni/urdf/mesh/end_effector_fork.dae" scale="1 1 1"/>
-        </geometry>
-      </visual>
-    </link>
-    <!-- Mount fork to the flange -->
-    <joint name="ee_mount_to_fork" type="fixed">
-      <parent link="ee_mount"/>
-      <child link="fork"/>
-      <origin xyz="0 0 0" rpy="0 0 0"/>
-    </joint>
-    <!-- Contact point for the fork tips -->
-    <joint name="fork_to_ee_contact" type="fixed">
-      <parent link="fork"/>
-      <child link="ee_contact"/>
-      <origin xyz="0 0 0.104" rpy="0 0 0"/>
-    </joint>
+    <xacro:fork_end_effector ee_mount_link="ee_mount"/>
   </xacro:if>
   <!-- ############# Ball tool ############# -->

Commit message: [urdf]: create ball_ee.xacro and put most contents from the main file into it
Signed-off-by: Jinjie Li <45286479+Li-Jinjie@users.noreply.github.com>

File: robots/beetle_omni/urdf/beetle_art_omni.urdf.xacro (robot description, xacro)
@@ -198,30 +198,7 @@
   </xacro:if>
   <!-- ############# Ball tool ############# -->
+  <xacro:include filename="$(find beetle_omni)/urdf/effectors/ball_ee.xacro"/>
   <xacro:if value="${end_effector == 'ball'}">
-    <link name="ball">
-      <inertial>
-        <origin xyz="0.00000000 0.08052689 0.00000000" rpy="0 0 0"/>
-        <mass value="0.1030"/>
-        <inertia
-                ixx="0.00020646" iyy="0.00008167" izz="0.00020646"
-                ixy="0.00000000" ixz="0.00000000" iyz="0.00000000"/>
-      </inertial>
-      <visual>
-        <geometry>
-          <mesh filename="package://beetle_omni/urdf/mesh/end_effector_ball.dae" scale="1 1 1"/>
-        </geometry>
-      </visual>
-    </link>
-    <joint name="ee_mount_to_ball" type="fixed">
-      <parent link="ee_mount"/>
-      <child link="ball"/>
-      <origin xyz="0 0 0" rpy="0 0 0"/>
-    </joint>
-    <!-- Contact point at the ball’s center -->
-    <joint name="ball_to_ee_contact" type="fixed">
-      <parent link="ball"/>
-      <child link="ee_contact"/>
-      <origin xyz="0 0 0.11" rpy="0 0 0"/>
-    </joint>
+    <xacro:ball_end_effector ee_mount_link="ee_mount"/>
   </xacro:if>
   <!-- ############# Sensor‑ball tool ############# -->

Commit message: [urdf]: create force_sensor_ball_ee.xacro and put most contents from the main file into it
Signed-off-by: Jinjie Li <45286479+Li-Jinjie@users.noreply.github.com>

File: robots/beetle_omni/urdf/beetle_art_omni.urdf.xacro (robot description, xacro)
@@ -203,52 +203,7 @@
   </xacro:if>
   <!-- ############# Sensor‑ball tool ############# -->
+  <xacro:include filename="$(find beetle_omni)/urdf/effectors/force_sensor_ball_ee.xacro"/>
   <xacro:if value="${end_effector == 'sensor_ball'}">
-    <!-- Wrench sensor -->
-    <link name="wrench_sensor">
-      <inertial>
-        <origin xyz="0.00000000 0.00000000 -0.01500000" rpy="0 0 0"/>
-        <mass value="0.285"/>
-        <inertia
-                ixx="0.00008773" iyy="0.00012377" izz="0.00016573"
-                ixy="0.00000000" ixz="0.00000328" iyz="0.00000000"/>
-      </inertial>
-      <visual>
-        <geometry>
-          <mesh filename="package://beetle_omni/urdf/mesh/wrench_sensor_pfs055ya501u6.dae" scale="1 1 1"/>
-        </geometry>
-      </visual>
-    </link>
-    <joint name="ee_mount_to_sensor" type="fixed">
-      <parent link="ee_mount"/>
-      <child link="wrench_sensor"/>
-      <origin xyz="0 0 0.031" rpy="0 0 0"/>
-    </joint>
-    <!-- Ball attached to the sensor -->
-    <link name="ball">
-      <!-- (same as plain ball) -->
-      <inertial>
-        <origin xyz="0.00000000 0.08052689 0.00000000" rpy="0 0 0"/>
-        <mass value="0.1030"/>
-        <inertia
-                ixx="0.00020646" iyy="0.00008167" izz="0.00020646"
-                ixy="0.00000000" ixz="0.00000000" iyz="0.00000000"/>
-      </inertial>
-      <visual>
-        <geometry>
-          <mesh filename="package://beetle_omni/urdf/mesh/end_effector_ball.dae" scale="1 1 1"/>
-        </geometry>
-      </visual>
-    </link>
-    <joint name="sensor_to_ball" type="fixed">
-      <parent link="wrench_sensor"/>
-      <child link="ball"/>
-      <origin xyz="0 0 0" rpy="0 0 0"/>
-    </joint>
-    <!-- Contact point at ball tip -->
-    <joint name="ball_to_ee_contact" type="fixed">
-      <parent link="ball"/>
-      <child link="ee_contact"/>
-      <origin xyz="0 0 0.11" rpy="0 0 0"/>
-    </joint>
+    <xacro:force_sensor_ball_end_effector ee_mount_link="ee_mount"/>
   </xacro:if>
   <!-- ############# Brush tool ############# -->
