Commit message: [urdf]: make robot_ns a general interface for all end effectors
Signed-off-by: Jinjie Li <45286479+Li-Jinjie@users.noreply.github.com>

File: robots/beetle_omni/urdf/beetle_art_omni.urdf.xacro (robot description, xacro)
@@ -195,20 +195,20 @@
   <xacro:include filename="$(find beetle_omni)/urdf/effectors/fork_ee.xacro"/>
   <xacro:if value="${end_effector == 'fork'}">
-    <xacro:fork_end_effector ee_mount_link="ee_mount"/>
+    <xacro:fork_end_effector ee_mount_link="ee_mount" robot_ns="${robot_name}"/>
   </xacro:if>
   <!-- ############# Ball tool ############# -->
   <xacro:include filename="$(find beetle_omni)/urdf/effectors/ball_ee.xacro"/>
   <xacro:if value="${end_effector == 'ball'}">
-    <xacro:ball_end_effector ee_mount_link="ee_mount"/>
+    <xacro:ball_end_effector ee_mount_link="ee_mount" robot_ns="${robot_name}"/>
   </xacro:if>
   <!-- ############# Sensor‑ball tool ############# -->
   <xacro:include filename="$(find beetle_omni)/urdf/effectors/force_sensor_ball_ee.xacro"/>
   <xacro:if value="${end_effector == 'sensor_ball'}">
-    <xacro:force_sensor_ball_end_effector ee_mount_link="ee_mount"/>
+    <xacro:force_sensor_ball_end_effector ee_mount_link="ee_mount" robot_ns="${robot_name}"/>
   </xacro:if>
   <!-- ############# Brush tool ############# -->
   <xacro:include filename="$(find beetle_omni)/urdf/effectors/brush_ee.xacro"/>
   <xacro:if value="${end_effector == 'brush'}">
-    <xacro:brush_end_effector ee_mount_link="ee_mount"/>
+    <xacro:brush_end_effector ee_mount_link="ee_mount" robot_ns="${robot_name}"/>
   </xacro:if>
   <!-- ############# DJI OSMO Action 4 ############# -->

File: robots/beetle_omni/urdf/effectors/ball_ee.xacro (robot description, xacro)
@@ -6,5 +6,5 @@
       ee_mount_link : The base link that the ball tool is mounted to (e.g. "ee_mount").
   -->
-  <xacro:macro name="ball_end_effector" params="ee_mount_link">
+  <xacro:macro name="ball_end_effector" params="ee_mount_link robot_ns">
     <!-- 1) Ball tool geometry and inertia -->
     <link name="ball">

File: robots/beetle_omni/urdf/effectors/brush_ee.xacro (robot description, xacro)
@@ -6,5 +6,5 @@
       ee_mount_link : The base link connected to the end-effector (e.g. "ee_mount").
   -->
-  <xacro:macro name="brush_end_effector" params="ee_mount_link">
+  <xacro:macro name="brush_end_effector" params="ee_mount_link robot_ns">
     <!-- 1) Main brush body link and joint -->
     <link name="brush">
@@ -26,5 +26,5 @@
           <!-- You can reuse the same mesh for collision or a simplified one -->
           <mesh filename="package://beetle_omni/urdf/mesh/end_effector_brush.dae"
-                      scale="1 1 1"/>
+                scale="1 1 1"/>
         </geometry>
       </collision>
@@ -32,5 +32,5 @@
     <joint name="ee_mount_to_brush" type="fixed">
       <parent link="${ee_mount_link}"/>
-      <child  link="brush"/>
+      <child link="brush"/>
       <origin xyz="0 0 0" rpy="0 0 0"/>
     </joint>
@@ -39,9 +39,9 @@
     <joint name="brush_to_ee_contact" type="fixed">
       <parent link="brush"/>
-      <child  link="ee_contact"/>
+      <child link="ee_contact"/>
       <origin xyz="0 0 0.144" rpy="0 0 0"/>
     </joint>
     <!--  3) Attach the ark_flow_sensor  -->
-    <xacro:ark_flow_sensor parent_link="ee_mount"/>
+    <xacro:ark_flow_sensor parent_link="ee_mount" robot_ns="${robot_ns}"/>
   </xacro:macro>
   <!--

File: robots/beetle_omni/urdf/effectors/force_sensor_ball_ee.xacro (robot description, xacro)
@@ -8,5 +8,5 @@
       ee_mount_link : The base link that the sensor-ball tool is mounted to (e.g. "ee_mount").
   -->
-  <xacro:macro name="force_sensor_ball_end_effector" params="ee_mount_link">
+  <xacro:macro name="force_sensor_ball_end_effector" params="ee_mount_link robot_ns">
     <!-- 1) Wrench sensor link -->
     <link name="wrench_sensor">
@@ -49,5 +49,5 @@
       ee_contact is assumed to be defined elsewhere.
     -->
-    <xacro:ball_end_effector ee_mount_link="wrench_sensor"/>
+    <xacro:ball_end_effector ee_mount_link="wrench_sensor" robot_ns="${robot_name}"/>
   </xacro:macro>
 </robot>

File: robots/beetle_omni/urdf/effectors/fork_ee.xacro (robot description, xacro)
@@ -6,5 +6,5 @@
       ee_mount_link : The base link that the fork tool is mounted to (e.g. "ee_mount").
   -->
-  <xacro:macro name="fork_end_effector" params="ee_mount_link">
+  <xacro:macro name="fork_end_effector" params="ee_mount_link robot_ns">
     <!-- 1) Fork tool geometry and inertia -->
     <link name="fork">

Commit message: [omni][urdf]: add none option for no effector.
Signed-off-by: Jinjie Li <45286479+Li-Jinjie@users.noreply.github.com>

File: robots/beetle_omni/urdf/beetle_art_omni.urdf.xacro (robot description, xacro)
@@ -198,5 +198,5 @@
   <xacro:property name="end_effector" value="$(arg end_effector)"/>
   <xacro:if value="${end_effector != 'fork' and end_effector != 'ball' and end_effector != 'sensor_ball'
-  and end_effector != 'brush' and end_effector != 'osmo'}">
+  and end_effector != 'brush' and end_effector != 'osmo' and end_effector != 'none'}">
     <xacro:error>Invalid end_effector type: ${end_effector}. Must be one of: fork, ball, sensor_ball, brush, osmo.</xacro:error>
   </xacro:if>
@@ -210,4 +210,13 @@
   <!-- Tool‑agnostic contact frame (pose set inside each branch) -->
   <link name="ee_contact"/>
+  <!-- ############# None ############# -->
+  <xacro:if value="${end_effector == 'none'}">
+    <!-- atach ee_contact to ee_mount -->
+    <joint name="ee_mount_to_ee_contact" type="fixed">
+      <parent link="ee_mount"/>
+      <child link="ee_contact"/>
+      <origin xyz="0 0 0" rpy="0 0 0"/>
+    </joint>
+  </xacro:if>
   <!-- ############# Fork tool ############# -->
   <xacro:include filename="$(find beetle_omni)/urdf/effectors/fork_ee.xacro"/>
