Commit message: [effectors]: make ee_contact_link a parameter
Signed-off-by: Jinjie Li <45286479+Li-Jinjie@users.noreply.github.com>

File: robots/beetle_omni/urdf/dragon_ball.urdf.xacro (robot description, xacro)
@@ -194,9 +194,10 @@
   <xacro:dragon_ball_thrust_link self="4" rotor_direction="-1"/>
   <!-- ============ End‑Effector (EE) =============== -->
-  <!-- Select EE type:  fork | ball | sensor_ball | brush -->
+  <!-- Select EE type:  fork | ball | sensor_ball | brush | osmo | none -->
   <xacro:arg name="end_effector" default="fork"/>
   <xacro:property name="end_effector" value="$(arg end_effector)"/>
-  <xacro:if value="${end_effector != 'fork' and end_effector != 'ball' and end_effector != 'sensor_ball'
-  and end_effector != 'brush' and end_effector != 'osmo'}">
+  <xacro:if value="${end_effector != 'none' and end_effector != 'fork' and end_effector != 'ball' and end_effector != 'sensor_ball'
+  and end_effector != 'brush' and end_effector != 'osmo' and  end_effector != 'brush_short' and end_effector !='mouse'
+  and end_effector !='droplet_head'}">
     <xacro:error>Invalid end_effector type: ${end_effector}. Must be one of: fork, ball, sensor_ball, brush, osmo.</xacro:error>
   </xacro:if>
@@ -210,13 +211,51 @@
   <!-- Tool‑agnostic contact frame (pose set inside each branch) -->
   <link name="ee_contact"/>
+  <!-- +++++++++ EE bottom ++++++++++ -->
+  <xacro:arg name="end_effector_bottom" default="brush_short"/>
+  <xacro:property name="end_effector_bottom" value="$(arg end_effector_bottom)"/>
+  <xacro:if value="${end_effector_bottom != 'none' and end_effector_bottom != 'fork' and end_effector_bottom != 'ball' and end_effector_bottom != 'sensor_ball'
+  and end_effector_bottom != 'brush' and end_effector_bottom != 'brush_short' and end_effector_bottom !='mouse'
+  and end_effector_bottom !='droplet_tail'}">
+    <xacro:error>Invalid end_effector_bottom type: ${end_effector_bottom}. Must be one of: fork, ball, sensor_ball, brush, brush_short, mouse, droplet_tail, none.</xacro:error>
+  </xacro:if>
+  <!-- Fixed the flange that all tools attach to -->
+  <link name="ee_bottom_mount"/>
+  <joint name="body_to_ee_bottom_mount" type="fixed">
+    <parent link="main_body"/>
+    <child link="ee_bottom_mount"/>
+    <origin xyz="0 0 -0.062" rpy="0 3.1415926 0"/>
+  </joint>
+  <!-- Tool‑agnostic contact frame (pose set inside each branch) -->
+  <link name="ee_bottom_contact"/>
+  <!-- ############# None ############# -->
+  <xacro:if value="${end_effector == 'none'}">
+    <!-- attach ee_contact to ee_mount (top) -->
+    <joint name="ee_mount_to_ee_contact" type="fixed">
+      <parent link="ee_mount"/>
+      <child link="ee_contact"/>
+      <origin xyz="0 0 0" rpy="0 0 0"/>
+    </joint>
+    <!-- attach ee_bottom_contact to ee_bottom_mount -->
+    <joint name="ee_bottom_mount_to_ee_bottom_contact" type="fixed">
+      <parent link="ee_bottom_mount"/>
+      <child link="ee_bottom_contact"/>
+      <origin xyz="0 0 0" rpy="0 0 0"/>
+    </joint>
+  </xacro:if>
   <!-- ############# Fork tool ############# -->
   <xacro:include filename="$(find beetle_omni)/urdf/effectors/fork_ee.xacro"/>
   <xacro:if value="${end_effector == 'fork'}">
-    <xacro:fork_end_effector ee_mount_link="ee_mount" robot_ns="${robot_name}"/>
+    <xacro:fork_end_effector ee_mount_link="ee_mount" ee_contact_link="ee_contact" robot_ns="${robot_name}"/>
+  </xacro:if>
+  <xacro:if value="${end_effector_bottom == 'fork'}">
+    <xacro:fork_end_effector ee_mount_link="ee_bottom_mount" ee_contact_link="ee_bottom_contact" robot_ns="${robot_name}"/>
   </xacro:if>
   <!-- ############# Ball tool ############# -->
   <xacro:include filename="$(find beetle_omni)/urdf/effectors/ball_ee.xacro"/>
   <xacro:if value="${end_effector == 'ball'}">
-    <xacro:ball_end_effector ee_mount_link="ee_mount" robot_ns="${robot_name}"/>
+    <xacro:ball_end_effector ee_mount_link="ee_mount" ee_contact_link="ee_contact" robot_ns="${robot_name}"/>
+  </xacro:if>
+  <xacro:if value="${end_effector_bottom == 'ball'}">
+    <xacro:ball_end_effector ee_mount_link="ee_bottom_mount" ee_contact_link="ee_bottom_contact" robot_ns="${robot_name}"/>
   </xacro:if>
   <!-- ############# Sensor‑ball tool ############# -->
@@ -225,13 +264,44 @@
     <xacro:force_sensor_ball_end_effector ee_mount_link="ee_mount" robot_ns="${robot_name}"/>
   </xacro:if>
+  <xacro:if value="${end_effector_bottom == 'sensor_ball'}">
+    <xacro:force_sensor_ball_end_effector ee_mount_link="ee_bottom_mount" robot_ns="${robot_name}"/>
+  </xacro:if>
   <!-- ############# Brush tool ############# -->
   <xacro:include filename="$(find beetle_omni)/urdf/effectors/brush_ee.xacro"/>
   <xacro:if value="${end_effector == 'brush'}">
-    <xacro:brush_end_effector ee_mount_link="ee_mount" robot_ns="${robot_name}"/>
+    <xacro:brush_end_effector ee_mount_link="ee_mount" ee_contact_link="ee_contact" robot_ns="${robot_name}"/>
+  </xacro:if>
+  <xacro:if value="${end_effector_bottom == 'brush'}">
+    <xacro:brush_end_effector ee_mount_link="ee_bottom_mount" ee_contact_link="ee_bottom_contact" robot_ns="${robot_name}"/>
   </xacro:if>
   <!-- ############# DJI OSMO Action 4 ############# -->
   <xacro:include filename="$(find beetle_omni)/urdf/effectors/osmo_cam_ee.xacro"/>
   <xacro:if value="${end_effector == 'osmo'}">
-    <xacro:osmo_end_effector ee_mount_link="ee_mount" robot_ns="${robot_name}"/>
+    <xacro:osmo_end_effector ee_mount_link="ee_mount" ee_contact_link="ee_contact" robot_ns="${robot_name}"/>
+  </xacro:if>
+  <!-- ############# Short Brush tool ############# -->
+  <xacro:include filename="$(find beetle_omni)/urdf/effectors/brush_short_ee.xacro"/>
+  <xacro:if value="${end_effector == 'brush_short'}">
+    <xacro:brush_short_end_effector ee_mount_link="ee_mount" ee_contact_link="ee_contact" robot_ns="${robot_name}"/>
+  </xacro:if>
+  <xacro:if value="${end_effector_bottom == 'brush_short'}">
+    <xacro:brush_short_end_effector ee_mount_link="ee_bottom_mount" ee_contact_link="ee_bottom_contact" robot_ns="${robot_name}"/>
+  </xacro:if>
+  <!-- ############# Mouse tool ############# -->
+  <xacro:include filename="$(find beetle_omni)/urdf/effectors/mouse_ee.xacro"/>
+  <xacro:if value="${end_effector == 'mouse'}">
+    <xacro:mouse_end_effector ee_mount_link="ee_mount" ee_contact_link="ee_contact" robot_ns="${robot_name}"/>
+  </xacro:if>
+  <xacro:if value="${end_effector_bottom == 'mouse'}">
+    <xacro:mouse_end_effector ee_mount_link="ee_bottom_mount" ee_contact_link="ee_bottom_contact" robot_ns="${robot_name}"/>
+  </xacro:if>
+  <!-- ############# Droplet ############# -->
+  <xacro:include filename="$(find beetle_omni)/urdf/effectors/droplet_head_ee.xacro"/>
+  <xacro:if value="${end_effector == 'droplet_head'}">
+    <xacro:droplet_head_end_effector ee_mount_link="ee_mount" ee_contact_link="ee_contact" robot_ns="${robot_name}"/>
+  </xacro:if>
+  <xacro:include filename="$(find beetle_omni)/urdf/effectors/droplet_tail_ee.xacro"/>
+  <xacro:if value="${end_effector_bottom == 'droplet_tail'}">
+    <xacro:droplet_tail_end_effector ee_mount_link="ee_bottom_mount" ee_contact_link="ee_bottom_contact" robot_ns="${robot_name}"/>
   </xacro:if>
 </robot>

File: robots/beetle_omni/urdf/effectors/ball_ee.xacro (robot description, xacro)
@@ -4,7 +4,9 @@
     Macro: ball_end_effector
     params:
-      ee_mount_link : The base link that the ball tool is mounted to (e.g. "ee_mount").
+      ee_mount_link : The base link that the ball tool is mounted to (e.g. "ee_mount" or "ee_bottom_mount").
+      ee_contact_link : The contact link name (e.g. "ee_contact" or "ee_bottom_contact").
+      robot_ns      : ROS namespace
   -->
-  <xacro:macro name="ball_end_effector" params="ee_mount_link robot_ns">
+  <xacro:macro name="ball_end_effector" params="ee_mount_link ee_contact_link robot_ns">
     <!-- 1) Ball tool geometry and inertia -->
     <link name="ball">
@@ -40,8 +42,8 @@
     </joint>
     <!-- 3) Contact frame at the ball's contact point -->
-    <!-- ee_contact is assumed to be defined elsewhere -->
+    <!-- ee_contact_link is passed as parameter -->
     <joint name="ball_to_ee_contact" type="fixed">
       <parent link="ball"/>
-      <child link="ee_contact"/>
+      <child link="${ee_contact_link}"/>
       <origin xyz="0 0 0.11" rpy="0 0 0"/>
     </joint>

File: robots/beetle_omni/urdf/effectors/brush_ee.xacro (robot description, xacro)
@@ -4,7 +4,8 @@
     Macro: brush_end_effector
     params:
-      ee_mount_link : The base link connected to the end-effector (e.g. "ee_mount").
+      ee_mount_link : The base link connected to the end-effector (e.g. "ee_mount" or "ee_bottom_mount").
+      robot_ns      : ROS namespace
   -->
-  <xacro:macro name="brush_end_effector" params="ee_mount_link robot_ns">
+  <xacro:macro name="brush_end_effector" params="ee_mount_link ee_contact_link robot_ns">
     <!-- 1) Main brush body link and joint -->
     <link name="brush">
@@ -36,8 +37,8 @@
     </joint>
     <!-- 2) Contact frame at the bristle tip, required by the outer framework -->
-    <!-- ee_contact is assumed to be defined elsewhere -->
+    <!-- ee_contact_link is passed as parameter -->
     <joint name="brush_to_ee_contact" type="fixed">
       <parent link="brush"/>
-      <child link="ee_contact"/>
+      <child link="${ee_contact_link}"/>
       <origin xyz="0 0 0.144" rpy="0 0 0"/>
     </joint>

File: robots/beetle_omni/urdf/effectors/brush_short_ee.xacro (robot description, xacro)
@@ -4,7 +4,8 @@
     Macro: brush_short_end_effector
     params:
-      ee_mount_link : The base link connected to the end-effector (e.g. "ee_mount").
+      ee_mount_link : The base link connected to the end-effector (e.g. "ee_mount" or "ee_bottom_mount").
+      robot_ns      : ROS namespace
   -->
-  <xacro:macro name="brush_short_end_effector" params="ee_mount_link robot_ns">
+  <xacro:macro name="brush_short_end_effector" params="ee_mount_link ee_contact_link robot_ns">
     <!-- 1) Main brush body link and joint -->
     <link name="brush_short">
@@ -36,8 +37,8 @@
     </joint>
     <!-- 2) Contact frame at the bristle tip, required by the outer framework -->
-    <!-- ee_contact is assumed to be defined elsewhere -->
+    <!-- ee_contact_link is passed as parameter -->
     <joint name="brush_to_ee_contact" type="fixed">
       <parent link="brush_short"/>
-      <child link="ee_contact"/>
+      <child link="${ee_contact_link}"/>
       <origin xyz="0 0 0.076" rpy="0 0 0"/>
     </joint>

File: robots/beetle_omni/urdf/effectors/droplet_head_ee.xacro (robot description, xacro)
@@ -4,7 +4,8 @@
     Macro: droplet_head_end_effector
     params:
-      ee_mount_link : The base link connected to the end-effector (e.g. "ee_mount").
+      ee_mount_link : The base link connected to the end-effector (e.g. "ee_mount" or "ee_bottom_mount").
+      robot_ns      : ROS namespace
   -->
-  <xacro:macro name="droplet_head_end_effector" params="ee_mount_link robot_ns">
+  <xacro:macro name="droplet_head_end_effector" params="ee_mount_link ee_contact_link robot_ns">
     <!-- 1) Main body link and joint -->
     <link name="droplet_head">
@@ -36,8 +37,8 @@
     </joint>
     <!-- 2) Contact frame at the bristle tip, required by the outer framework -->
-    <!-- ee_contact is assumed to be defined elsewhere -->
+    <!-- ee_contact_link is passed as parameter -->
     <joint name="droplet_head_to_ee_contact" type="fixed">
       <parent link="droplet_head"/>
-      <child link="ee_contact"/>
+      <child link="${ee_contact_link}"/>
       <origin xyz="0 0 0.042" rpy="0 0 0"/>
     </joint>

File: robots/beetle_omni/urdf/effectors/droplet_tail_ee.xacro (robot description, xacro)
@@ -4,7 +4,8 @@
     Macro: droplet_tail_end_effector
     params:
-      ee_mount_link : The base link connected to the end-effector (e.g. "ee_mount").
+      ee_mount_link : The base link connected to the end-effector (e.g. "ee_mount" or "ee_bottom_mount").
+      robot_ns      : ROS namespace
   -->
-  <xacro:macro name="droplet_tail_end_effector" params="ee_mount_link robot_ns">
+  <xacro:macro name="droplet_tail_end_effector" params="ee_mount_link ee_contact_link robot_ns">
     <!-- 1) Main body link and joint -->
     <link name="droplet_tail">
@@ -36,8 +37,8 @@
     </joint>
     <!-- 2) Contact frame at the bristle tip, required by the outer framework -->
-    <!-- ee_contact is assumed to be defined elsewhere -->
+    <!-- ee_contact_link is passed as parameter -->
     <joint name="droplet_tail_to_ee_contact" type="fixed">
       <parent link="droplet_tail"/>
-      <child link="ee_contact"/>
+      <child link="${ee_contact_link}"/>
       <origin xyz="0 0 0.192" rpy="0 0 0"/>
     </joint>

File: robots/beetle_omni/urdf/effectors/force_sensor_ball_ee.xacro (robot description, xacro)
@@ -6,7 +6,8 @@
     Macro: force_sensor_ball_end_effector
     params:
-      ee_mount_link : The base link that the sensor-ball tool is mounted to (e.g. "ee_mount").
+      ee_mount_link : The base link that the sensor-ball tool is mounted to (e.g. "ee_mount" or "ee_bottom_mount").
+      robot_ns      : ROS namespace
   -->
-  <xacro:macro name="force_sensor_ball_end_effector" params="ee_mount_link robot_ns">
+  <xacro:macro name="force_sensor_ball_end_effector" params="ee_mount_link ee_contact_link robot_ns">
     <!-- 1) Wrench sensor link -->
     <link name="wrench_sensor">
@@ -46,8 +47,8 @@
         - create link "ball"
         - add joint "ee_mount_to_ball" from wrench_sensor to ball
-        - add joint "ball_to_ee_contact" from ball to ee_contact
-      ee_contact is assumed to be defined elsewhere.
+        - add joint "ball_to_ee_contact" from ball to ee_contact_link
+      ee_contact_link is passed as parameter.
     -->
-    <xacro:ball_end_effector ee_mount_link="wrench_sensor" robot_ns="${robot_name}"/>
+    <xacro:ball_end_effector ee_mount_link="wrench_sensor" ee_contact_link="${ee_contact_link}" robot_ns="${robot_name}"/>
   </xacro:macro>
 </robot>

File: robots/beetle_omni/urdf/effectors/fork_ee.xacro (robot description, xacro)
@@ -4,7 +4,8 @@
     Macro: fork_end_effector
     params:
-      ee_mount_link : The base link that the fork tool is mounted to (e.g. "ee_mount").
+      ee_mount_link : The base link that the fork tool is mounted to (e.g. "ee_mount" or "ee_bottom_mount").
+      robot_ns      : ROS namespace
   -->
-  <xacro:macro name="fork_end_effector" params="ee_mount_link robot_ns">
+  <xacro:macro name="fork_end_effector" params="ee_mount_link ee_contact_link robot_ns">
     <!-- 1) Fork tool geometry and inertia -->
     <link name="fork">
@@ -38,8 +39,8 @@
     </joint>
     <!-- 3) Contact frame at the fork tips, required by the outer framework -->
-    <!-- ee_contact is assumed to be defined elsewhere -->
+    <!-- ee_contact_link is passed as parameter -->
     <joint name="fork_to_ee_contact" type="fixed">
       <parent link="fork"/>
-      <child link="ee_contact"/>
+      <child link="${ee_contact_link}"/>
       <origin xyz="0 0 0.104" rpy="0 0 0"/>
     </joint>

File: robots/beetle_omni/urdf/effectors/mouse_ee.xacro (robot description, xacro)
@@ -4,7 +4,8 @@
     Macro: mouse_end_effector
     params:
-      ee_mount_link : The base link connected to the end-effector (e.g. "ee_mount").
+      ee_mount_link : The base link connected to the end-effector (e.g. "ee_mount" or "ee_bottom_mount").
+      robot_ns      : ROS namespace
   -->
-  <xacro:macro name="mouse_end_effector" params="ee_mount_link robot_ns">
+  <xacro:macro name="mouse_end_effector" params="ee_mount_link ee_contact_link robot_ns">
     <!-- 1) Main body link and joint -->
     <link name="mouse">
@@ -36,8 +37,8 @@
     </joint>
     <!-- 2) Contact frame at the bristle tip, required by the outer framework -->
-    <!-- ee_contact is assumed to be defined elsewhere -->
+    <!-- ee_contact_link is passed as parameter -->
     <joint name="mouse_to_ee_contact" type="fixed">
       <parent link="mouse"/>
-      <child link="ee_contact"/>
+      <child link="${ee_contact_link}"/>
       <origin xyz="0 0 0.055" rpy="0 0 0"/>
     </joint>

File: robots/beetle_omni/urdf/effectors/osmo_cam_ee.xacro (robot description, xacro)
@@ -4,8 +4,8 @@
     Macro: osmo_end_effector
     params:
-      ee_mount_link : The base link connected to the end-effector. (e.g., "ee_mount")
-      robot_ns    : ROS namespace (e.g. "beetle1"). Can be "".
+      ee_mount_link : The base link connected to the end-effector. (e.g., "ee_mount" or "ee_bottom_mount")
+      robot_ns      : ROS namespace (e.g. "beetle1"). Can be "".
   -->
-  <xacro:macro name="osmo_end_effector" params="ee_mount_link robot_ns">
+  <xacro:macro name="osmo_end_effector" params="ee_mount_link ee_contact_link robot_ns">
     <!-- 1) OSMO link and joint -->
     <link name="osmo">
@@ -33,5 +33,5 @@
     <joint name="osmo_to_ee_contact" type="fixed">
       <parent link="osmo"/>
-      <child link="ee_contact"/>
+      <child link="${ee_contact_link}"/>
       <origin xyz="0 0 0.045" rpy="0 0 0"/>
     </joint>

Commit message: [ball][urdf]: update the motor info based on config
Signed-off-by: Jinjie Li <45286479+Li-Jinjie@users.noreply.github.com>

File: robots/beetle_omni/urdf/dragon_ball.urdf.xacro (robot description, xacro)
@@ -4,6 +4,6 @@
   <baselink name="fc" />
   <thrust_link name="thrust" />
-  <m_f_rate value="-0.0165" /> <!-- drag torque rate -->
-  <xacro:property name="max_force" value="30.0" /> <!-- [N] -->
+  <m_f_rate value="-0.0112" /> <!-- drag torque rate -->
+  <xacro:property name="max_force" value="15.0" /> <!-- [N] -->
   <xacro:property name="min_force" value="1.0" /> <!-- [N] -->
   <!-- friction -->

Commit message: [ball][bi][urdf]: update part of parameters same with dragon_ball
Signed-off-by: Jinjie Li <45286479+Li-Jinjie@users.noreply.github.com>

File: robots/beetle_omni/urdf/dragon_ball.urdf.xacro (robot description, xacro)
@@ -26,9 +26,9 @@
     <link name="main_body">
       <inertial>
-        <origin xyz="-0.00058556 0.00011136 0.00444799" rpy="0 0 0"/>
+        <origin xyz="-0.00057669 0.00011619 0.00444799" rpy="0 0 0"/>
         <mass value="1.1340"/>
         <inertia
-            ixx="0.00358514" iyy="0.00354587" izz="0.00357606"
-            ixy="-0.00000033" ixz="-0.00005534" iyz="0.00000798"/>
+            ixx="0.00358540" iyy="0.00354562" izz="0.00357607"
+            ixy="-0.00000017" ixz="-0.00005461" iyz="0.00000844"/>
       </inertial>
       <visual>

File: robots/beetle_omni/urdf/dragon_ball_bi.urdf.xacro (robot description, xacro)
@@ -26,9 +26,9 @@
     <link name="main_body">
       <inertial>
-        <origin xyz="-0.00058556 0.00011136 0.00444799" rpy="0 0 0"/>
+        <origin xyz="-0.00057669 0.00011619 0.00444799" rpy="0 0 0"/>
         <mass value="1.1340"/>
         <inertia
-            ixx="0.00358514" iyy="0.00354587" izz="0.00357606"
-            ixy="-0.00000033" ixz="-0.00005534" iyz="0.00000798"/>
+            ixx="0.00358540" iyy="0.00354562" izz="0.00357607"
+            ixy="-0.00000017" ixz="-0.00005461" iyz="0.00000844"/>
       </inertial>
       <visual>

Commit message: [ball][urdf]: add some h_flow sensors
Signed-off-by: Jinjie Li <45286479+Li-Jinjie@users.noreply.github.com>

File: robots/beetle_omni/urdf/dragon_ball.urdf.xacro (robot description, xacro)
@@ -1,4 +1,5 @@
 <?xml version="1.0"?>
 <robot xmlns:xacro="http://www.ros.org/wiki/xacro" name="dragon_ball_link" >
+  <xacro:include filename="$(find beetle_omni)/urdf/sensors/h_flow.xacro"/>
   <!-- general attribute -->
   <baselink name="fc" />
@@ -20,5 +21,5 @@
   </xacro:macro>
   <!-- robot -->
-  <xacro:macro name="dragon_ball_center_link" params="child1 child2 child3 child4">
+  <xacro:macro name="dragon_ball_center_link" params="child1 child2 child3 child4 has_h_flow">
     ## dummy
     <link name="root"/>
@@ -90,4 +91,12 @@
     <xacro:dummy_rotor_arm id = "${child3}" x = "-0.08231" y="-0.08231" z = "0.0175" yaw = "${pi*5.0/4.0}"/>
     <xacro:dummy_rotor_arm id = "${child4}" x = "0.08231" y="-0.08231" z = "0.0175" yaw = "${-pi*1.0/4.0}"/>
+    <xacro:if value="${has_h_flow}">
+      <xacro:h_flow_sensor name="h_flow_1" parent_link="main_body" robot_ns="${robot_name}" xyz="0.08357 0 0.104" rpy="0 0 0"/>
+      <xacro:h_flow_sensor name="h_flow_2" parent_link="main_body" robot_ns="${robot_name}" xyz="0.06377 0 0.021" rpy="0 1.570796 0"/>
+      <xacro:h_flow_sensor name="h_flow_3" parent_link="main_body" robot_ns="${robot_name}" xyz="0 0.06377 0.021" rpy="0 1.570796 1.570796"/>
+      <xacro:h_flow_sensor name="h_flow_4" parent_link="main_body" robot_ns="${robot_name}" xyz="-0.06377 0 0.021" rpy="0 1.570796 3.141592"/>
+      <xacro:h_flow_sensor name="h_flow_5" parent_link="main_body" robot_ns="${robot_name}" xyz="0 -0.06377 0.021" rpy="0 1.570796 -1.570796"/>
+      <xacro:h_flow_sensor name="h_flow_6" parent_link="main_body" robot_ns="${robot_name}" xyz="-0.08357 0 -0.062" rpy="3.141592 0 0"/>
+    </xacro:if>
     <xacro:friction self="main_body"/>
   </xacro:macro>
@@ -188,5 +197,6 @@
   <xacro:arg name="robot_name" default="dragon-ball" />
   <xacro:property name="robot_name" value="$(arg robot_name)"/>
-  <xacro:dragon_ball_center_link child1="1" child2="2" child3="3" child4="4"/>
+  <xacro:arg name="has_h_flow" default="false" />
+  <xacro:dragon_ball_center_link child1="1" child2="2" child3="3" child4="4" has_h_flow="$(arg has_h_flow)"/>
   <xacro:dragon_ball_thrust_link self="1" rotor_direction="1"/>
   <xacro:dragon_ball_thrust_link self="2" rotor_direction="-1"/>
