Commit message: [ball][bi][urdf]: modify the frame to make if possible to take off. But the oscillation is quite high, don't know why.
Signed-off-by: Jinjie Li <45286479+Li-Jinjie@users.noreply.github.com>

File: robots/beetle_omni/urdf/dragon_ball_bi.urdf.xacro (robot description, xacro)
@@ -48,5 +48,5 @@
       <parent link="root"/>
       <child link="main_body"/>
-      <origin rpy="0 0 0" xyz="0 0 0"/>
+      <origin rpy="0 0 0.78539816" xyz="0 0 0"/>
     </joint>
     <link name="fc">
@@ -62,5 +62,5 @@
     <joint name="fc_joint" type="fixed">
       <child link="fc"/>
-      <parent link="main_body"/>
+      <parent link="root"/>
       <origin rpy="0 0 0" xyz="-0.0175 -0.0015 0.075"/>  # should be aligned with the position of IMU
     </joint>

Commit message: [ball][bi][urdf]: fix the bug that only one frame can point to root link, otherwise KDL is wrong. Also fix the direction of root link to the front.
Signed-off-by: Jinjie Li <45286479+Li-Jinjie@users.noreply.github.com>

File: robots/beetle_omni/urdf/dragon_ball_bi.urdf.xacro (robot description, xacro)
@@ -48,5 +48,5 @@
       <parent link="root"/>
       <child link="main_body"/>
-      <origin rpy="0 0 0.78539816" xyz="0 0 0"/>
+      <origin rpy="0 0 -2.356194" xyz="0 0 0"/>
     </joint>
     <link name="fc">
@@ -62,6 +62,6 @@
     <joint name="fc_joint" type="fixed">
       <child link="fc"/>
-      <parent link="root"/>
-      <origin rpy="0 0 0" xyz="-0.0175 -0.0015 0.075"/>  # should be aligned with the position of IMU
+      <parent link="main_body"/>
+      <origin rpy="0 0 2.356194" xyz="-0.0175 -0.0015 0.075"/>  # should be aligned with the position of IMU
     </joint>
     ## rotor arm macro

Commit message: [ball][bi]: update the URDF and phy params based on the real robot

File: robots/beetle_omni/urdf/dragon_ball_bi.urdf.xacro (robot description, xacro)
@@ -48,5 +48,5 @@
       <parent link="root"/>
       <child link="main_body"/>
-      <origin rpy="0 0 -2.356194" xyz="0 0 0"/>
+      <origin rpy="0 0 0.785398" xyz="0 0 0"/>
     </joint>
     <link name="fc">
@@ -63,5 +63,5 @@
       <child link="fc"/>
       <parent link="main_body"/>
-      <origin rpy="0 0 2.356194" xyz="-0.0175 -0.0015 0.075"/>  # should be aligned with the position of IMU
+      <origin rpy="0 0 -0.785398" xyz="-0.01344 0.01131 0.075"/>  # should be aligned with the position of IMU
     </joint>
     ## rotor arm macro
